Commit message: cant use this cad

File: lab4/romeona_description/description/example_robot.urdf.xacro (robot description, xacro)
@@ -126,5 +126,5 @@
         <axis xyz="0 0 1"/>
         <limit lower="-1.57" upper="1.57" effort="0.5" velocity="0.5"/>
-        <dynamics damping="10" friction="10"/>
+        <dynamics damping="0" friction="0"/>
     </joint>
     <link name="link_3">
@@ -157,5 +157,5 @@
         <axis xyz="0 0 1"/>
         <limit lower="-1.57" upper="1.57" effort="1000" velocity="0.5"/>
-        <dynamics damping="10" friction="10"/>
+        <dynamics damping="0" friction="0"/>
     </joint>
     <joint name="joint_eff" type="fixed">

Commit message: marker

File: lab4/romeona_description/description/example_robot.urdf.xacro (robot description, xacro)
@@ -1,13 +1,4 @@
 <?xml version="1.0"?>
-<robot xmlns:xacro="http://www.ros.org/wiki/xacro"  name="romeona">
-<material name="Grey">
-  <color rgba="0.2 0.2 0.2 1.0"/>
-</material>
-<material name="Orange">
-  <color rgba="1.0 0.423529411765 0.0392156862745 1.0"/>
-</material>
-<material name="Blue">
-  <color rgba="0.5 0.7 1.0 1.0"/>
-</material>
+<robot xmlns:xacro="http://www.ros.org/wiki/xacro"  name="robot">
     <!-- This is an example of a URDF. -->
     <!-- As we move through the file, new things to note will be pointed out. -->
@@ -36,7 +27,4 @@
                 <mesh filename="file:///$(find romeona_description)/meshes/link_0.stl"/>
             </geometry>
-            <material name="Grey">
-                <color rgba="0.2 1 0.2 1"/>
-            </material>
         </visual>
         <collision>
@@ -49,7 +37,7 @@
         </collision>
         <inertial>
-            <origin xyz="0 0 0.05" rpy="0 0 0"/>
-            <mass value="4.91" />
-            <inertia ixx="0.03" ixy="0.0" ixz="0.0" iyy="0.03" iyz="0.0" izz="0.05" />
+            <origin xyz="0 0 .000914" rpy="0 0 0"/>
+            <mass value="0.16486" />
+            <inertia ixx="0.00015134507" ixy="0.0" ixz="0.0" iyy="0.00015134507" iyz="0.0" izz="0.00029194203" />
         </inertial>
     </link>
@@ -59,16 +47,21 @@
         <origin rpy="0 0 0" xyz="0 0 0"/>
         <axis xyz="0 0 1"/>
-        <limit lower="-3.14" upper="3.14" effort="1000" velocity="0.5"/>
+        <dynamics damping="0" friction="0"/>
+    </joint>
+    <joint name="joint_1" type="revolute">
+        <parent link="link_0"/>
+        <child link="link_1"/>
+        <origin rpy="0 0 0" xyz="0 0 0.135"/>
+        <axis xyz="0 0 1"/>
+        <limit lower="-3.14" upper="3.14" effort="0.5" velocity="0.5"/>
+        <dynamics damping="0" friction="0"/>
     </joint>
     <link name="link_1">
         <visual>
-            <origin xyz="0 0 0.0" rpy="0 0 0"/>
+            <origin rpy="0 0 3.14 " xyz="0 0 -0.125"/>
             <geometry>
                 <!-- <box size="2.5 1.5 0.1" /> -->
                 <mesh filename="file:///$(find romeona_description)/meshes/link_1.stl"/>
             </geometry>
-            <material name="Orange">
-                <color rgba="1.0 0.423529411765 0.0392156862745 1.0"/>
-            </material>
         </visual>
         <collision>
@@ -81,17 +74,17 @@
         </collision>
         <inertial>
-            <origin xyz="0 0 0.0" rpy="0 0 0"/>
-            <mass value="4.56" />
-            <inertia ixx="0.04" ixy="0.0" ixz="0.01" iyy="0.05" iyz="0.0" izz="0.02" />
+            <origin xyz="-0.00227 0 0.06038" rpy="0 0 0"/>
+            <mass value="0.33244" />
+            <inertia ixx="0.00050960520" ixy="0.0" ixz="-0.00004897127" iyy="0.00054096526" iyz="0.0" izz="0.00016177928" />
         </inertial>
     </link>
-    <joint name="joint_1" type="revolute">
-        <parent link="link_0"/>
-        <child link="link_1"/>
-        <origin rpy="0 0 0" xyz="0 0 0.3"/>
-        <axis xyz="0 0 1"/>
-        <limit lower="-3.14" upper="3.14" effort="1000" velocity="0.5"/>
-        <dynamics damping="0" friction="0"/>
-    </joint>
+  <joint name="joint_2" type="revolute">
+    <parent link="link_1"/>
+    <child link="link_2"/>
+    <origin rpy="1.57079632679   0 0" xyz="0.040 0 0"/>
+    <axis xyz="0 0 1"/>
+    <limit lower="-3.14" upper="3.14" effort="0.5" velocity="0.5"/>
+    <dynamics damping="0" friction="0"/>
+  </joint>
     <link name="link_2">
         <visual>
@@ -101,7 +94,4 @@
                 <mesh filename="file:///$(find romeona_description)/meshes/link_2.stl"/>
             </geometry>
-            <material name="Grey">
-                <color rgba="0.2 1 0.2 1"/>
-            </material>
         </visual>
         <collision>
@@ -115,17 +105,17 @@
         </collision>
         <inertial>
-            <origin xyz="0 0 0.0" rpy="0 0 0"/>
-            <mass value="3.56" />
-            <inertia ixx="0.01" ixy="0.0" ixz="0.0" iyy="0.04" iyz="0.0" izz="0.04" />
+            <origin xyz="0.07867 0 0.0" rpy="0 0 0"/>
+            <mass value="0.35295" />
+            <inertia ixx="0.000142422.27" ixy="0.0" ixz="0.0" iyy="0.00069087368" iyz="0.0" izz="0.00069536540" />
         </inertial>
     </link>
-    <joint name="joint_2" type="revolute">
-        <parent link="link_1"/>
-        <child link="link_2"/>
-        <origin rpy="1.57079632679   0 0" xyz="0.16 0 0"/>
+    <joint name="joint_3" type="revolute">
+        <parent link="link_2"/>
+        <child link="link_3"/>
+        <origin rpy="0 0 0" xyz="0.15 0 0"/>
         <axis xyz="0 0 1"/>
-        <limit lower="-1.57" upper="1.57" effort="0.5" velocity="0.5"/>
+        <limit lower="-3.14" upper="3.14" effort="0.5" velocity="0.5"/>
         <dynamics damping="0" friction="0"/>
-    </joint>
+      </joint>
     <link name="link_3">
         <visual>
@@ -134,7 +124,4 @@
                 <mesh filename="file:///$(find romeona_description)/meshes/link_3.stl"/>
             </geometry>
-            <material name="Orange">
-                <color rgba="1.0 0.423529411765 0.0392156862745 1.0"/>
-            </material>
         </visual>
         <collision>
@@ -146,25 +133,16 @@
         </collision>
         <inertial>
-            <origin xyz="0 0 0.0" rpy="0 0 0"/>
-            <mass value="1.23" />
-            <inertia ixx="0.00" ixy="0.0" ixz="0.0" iyy="0.00" iyz="0.0" izz="0.00" />
+            <origin xyz="0.04574 0 0.0" rpy="0 0 0"/>
+            <mass value="0.19651" />
+            <inertia ixx="0.00013273263" ixy="0.0" ixz="0.0" iyy="0.30209633" iyz="0.0" izz="0.00027662369" />
         </inertial>
     </link>
-    <joint name="joint_3" type="revolute">
-        <parent link="link_2"/>
-        <child link="link_3"/>
-        <origin rpy="0 0 0" xyz="0.35 0 0"/>
-        <axis xyz="0 0 1"/>
-        <limit lower="-1.57" upper="1.57" effort="1000" velocity="0.5"/>
-        <dynamics damping="0" friction="0"/>
-    </joint>
-    <joint name="joint_eff" type="fixed">
-        <parent link="link_3"/>
-        <child link="end_effector"/>
-        <origin rpy="1.57 0 1.57" xyz="0.16 0 0"/>
-        <axis xyz="0 0 1"/>
-    </joint>
-    <link name="end_effector">
-    </link>
+  <joint name="joint_eff" type="fixed">
+    <parent link="link_3"/>
+    <child link="end_effector"/>
+    <origin rpy="1.57 0 1.57" xyz="0.12 0 0"/>
+    <axis xyz="0 0 1"/>
+  </joint>
+    <link name="end_effector"/>
     <xacro:include filename="example_gazebo.xacro" />
 </robot>
