Commit message: complete

File: lab4/romeona_description/description/example_gazebo.xacro (robot description, xacro)
@@ -100,5 +100,5 @@
         <parent link="camera_link" />
         <child link="camera_link_optical" />
-    </joint>
+    </joint>[0.309,0.,0.134]
     <link name="camera_link_optical"></link> -->
     <!-- Add a gazebo tag for the ORIGINAL camera_link (but in the plugin we reference the optical frame so that ROS can orient things correctly) -->

File: lab4/romeona_description/description/example_robot.urdf.xacro (robot description, xacro)
@@ -1,4 +1,13 @@
 <?xml version="1.0"?>
 <robot xmlns:xacro="http://www.ros.org/wiki/xacro"  name="robot">
+<material name="Grey">
+  <color rgba="0.2 0.2 0.2 1.0"/>
+</material>
+<material name="Orange">
+  <color rgba="1.0 0.423529411765 0.0392156862745 1.0"/>
+</material>
+<material name="Blue">
+  <color rgba="0.5 0.7 1.0 1.0"/>
+</material>
     <!-- This is an example of a URDF. -->
     <!-- As we move through the file, new things to note will be pointed out. -->
@@ -27,4 +36,7 @@
                 <mesh filename="file:///$(find romeona_description)/meshes/link_0.stl"/>
             </geometry>
+            <material name="Grey">
+                <color rgba="0.2 1 0.2 1"/>
+            </material>
         </visual>
         <collision>
@@ -64,4 +76,7 @@
                 <mesh filename="file:///$(find romeona_description)/meshes/link_1.stl"/>
             </geometry>
+            <material name="Blue">
+                <color rgba="0.5 0.7 1.0 1.0"/>
+            </material>
         </visual>
         <collision>
@@ -94,4 +109,7 @@
                 <mesh filename="file:///$(find romeona_description)/meshes/link_2.stl"/>
             </geometry>
+            <material name="Grey">
+                <color rgba="0.2 1 0.2 1"/>
+            </material>
         </visual>
         <collision>
@@ -124,4 +142,7 @@
                 <mesh filename="file:///$(find romeona_description)/meshes/link_3.stl"/>
             </geometry>
+            <material name="Blue">
+                <color rgba="0.5 0.7 1.0 1.0"/>
+            </material>
         </visual>
         <collision>
